Commit message: Modify to enable "ros2 topic echo /scan" and "ros2 topic echo /odom"

File: urdf/barista_robot_model.urdf (robot description, URDF)
Before this commit: robot barista_robot, 7 links, 6 joints
Links:
- added link laser_scan_frame
Joints:
- added joint laser_scan_frame_joint: type fixed, parent laser_scanner_model, child laser_scan_frame, origin xyz=0 0 0.055 rpy=0 0 0, axis 0 0 0

Commit message: Add two caster wheels for stability of barista_robot

File: urdf/barista_robot_model.urdf (robot description, URDF)
Before this commit: robot barista_gazebo_robot, 8 links, 7 joints
Links:
- added link back_pitch_link, mass 0.06; collision sphere radius=0.0277; visual sphere radius=0.0277
- added link back_roll_link, mass 0.001; collision cylinder length=0.001 radius=0.0045000000000000005; visual cylinder length=0.001 radius=0.0045000000000000005
- added link back_yaw_link, mass 0.001; collision cylinder length=0.001 radius=0.0045000000000000005; visual cylinder length=0.001 radius=0.0045000000000000005
- added link front_pitch_link, mass 0.06; collision sphere radius=0.0277; visual sphere radius=0.0277
- added link front_roll_link, mass 0.001; collision cylinder length=0.001 radius=0.0045000000000000005; visual cylinder length=0.001 radius=0.0045000000000000005
- added link front_yaw_link, mass 0.001; collision cylinder length=0.001 radius=0.0045000000000000005; visual cylinder length=0.001 radius=0.0045000000000000005
Joints:
- added joint back_pitch_joint: type continuous, parent back_roll_link, child back_pitch_link, origin xyz=0 0 0 rpy=0 0 0, axis 0 1 0, limit effort=1000.0 velocity=100.0
- added joint back_roll_joint: type continuous, parent back_yaw_link, child back_roll_link, origin xyz=0 0 0 rpy=0 0 0, axis 1 0 0, limit effort=1000.0 velocity=100.0
- added joint back_yaw_joint: type continuous, parent main_body_link, child back_yaw_link, origin xyz=-0.13 0 0.0005 rpy=0 0 0, axis 0 0 1, limit effort=1000.0 velocity=100.0
- added joint front_pitch_joint: type continuous, parent front_roll_link, child front_pitch_link, origin xyz=0 0 0 rpy=0 0 0, axis 0 1 0, limit effort=1000.0 velocity=100.0
- added joint front_roll_joint: type continuous, parent front_yaw_link, child front_roll_link, origin xyz=0 0 0 rpy=0 0 0, axis 1 0 0, limit effort=1000.0 velocity=100.0
- added joint front_yaw_joint: type continuous, parent main_body_link, child front_yaw_link, origin xyz=0.13 0 0.0005 rpy=0 0 0, axis 0 0 1, limit effort=1000.0 velocity=100.0

Commit message: Update Fixing unstable robot status

File: urdf/barista_robot_model.urdf (robot description, URDF)
Before this commit: robot barista_robot, 14 links, 13 joints
Joints:
- joint back_yaw_joint: origin xyz=-0.13 0 0.0005 rpy=0 0 0 -> xyz=-0.13 0 0.0045 rpy=0 0 0
- joint front_yaw_joint: origin xyz=0.13 0 0.0005 rpy=0 0 0 -> xyz=0.13 0 0.0045 rpy=0 0 0
- joint left_wheel_joint: origin xyz=0.0 0.1 0.0352 rpy=0 0 0 -> xyz=0.0 0.1 0.0 rpy=0 0 0
- joint right_wheel_joint: origin xyz=0.0 -0.1 0.0352 rpy=0 0 0 -> xyz=0.0 -0.1 0.0 rpy=0 0 0

File: xacro/barista_robot_model.urdf.xacro (robot description, xacro)
@@ -50,5 +50,5 @@
     <xacro:wheel wheel_name="left_wheel"/>
     <joint name="left_wheel_joint" type="continuous">
-        <origin rpy="0 0 0" xyz="0.0 0.1 0.0352"/>
+        <origin rpy="0 0 0" xyz="0.0 0.1 0.0"/>
         <parent link="main_body_link"/>
         <child link="left_wheel"/>
@@ -73,5 +73,5 @@
     </gazebo>
     <joint name="right_wheel_joint" type="continuous">
-        <origin rpy="0 0 0" xyz="0.0 -0.1 0.0352"/>
+        <origin rpy="0 0 0" xyz="0.0 -0.1 0.0"/>
         <parent link="main_body_link"/>
         <child link="right_wheel"/>
@@ -84,18 +84,18 @@
     <link name="front_yaw_link">
         <visual>
-            <origin rpy="0 1.5707 1.5707" xyz="0 0 -0.0005"/>
-            <geometry>
-                <cylinder length="0.001" radius="0.0045000000000000005"/>
-            </geometry>
-            <material name="black"/>
-        </visual>
-        <collision>
-            <origin rpy="0 1.5707 1.5707" xyz="0 0 -0.0005"/>
-            <geometry>
-                <cylinder length="0.001" radius="0.0045000000000000005"/>
-            </geometry>
-        </collision>
-        <inertial>
-            <origin rpy="0 1.5707 1.5707" xyz="0 0 -0.0005"/>
+            <origin rpy="0 1.5707 1.5707" xyz="0.0 0 0.0"/>
+            <geometry>
+                <cylinder length="0.001" radius="0.0045000000000000005"/>
+            </geometry>
+            <material name="black"/>
+        </visual>
+        <collision>
+            <origin rpy="0 1.5707 1.5707" xyz="0.0 0 0.0"/>
+            <geometry>
+                <cylinder length="0.001" radius="0.0045000000000000005"/>
+            </geometry>
+        </collision>
+        <inertial>
+            <origin rpy="0 1.5707 1.5707" xyz="0.0 0 0.0"/>
             <mass value="0.001"/>
             <inertia ixx="5.145833333333334e-09" ixy="0" ixz="0" iyy="5.145833333333334e-09" iyz="0"
@@ -104,5 +104,5 @@
     </link>
     <joint name="front_yaw_joint" type="continuous">
-        <origin rpy="0 0 0" xyz="0.13 0 0.0005"/>
+        <origin rpy="0 0 0" xyz="0.13 0 0.0045"/>
         <parent link="main_body_link"/>
         <child link="front_yaw_link"/>
@@ -116,18 +116,18 @@
     <link name="front_roll_link">
         <visual>
-            <origin rpy="0 1.5707 1.5707" xyz="0 0 -0.0005"/>
-            <geometry>
-                <cylinder length="0.001" radius="0.0045000000000000005"/>
-            </geometry>
-            <material name="black"/>
-        </visual>
-        <collision>
-            <origin rpy="0 1.5707 1.5707" xyz="0 0 -0.0005"/>
-            <geometry>
-                <cylinder length="0.001" radius="0.0045000000000000005"/>
-            </geometry>
-        </collision>
-        <inertial>
-            <origin rpy="0 1.5707 1.5707" xyz="0 0 -0.0005"/>
+            <origin rpy="0 1.5707 1.5707" xyz="0 0 0"/>
+            <geometry>
+                <cylinder length="0.001" radius="0.0045000000000000005"/>
+            </geometry>
+            <material name="black"/>
+        </visual>
+        <collision>
+            <origin rpy="0 1.5707 1.5707" xyz="0 0 0"/>
+            <geometry>
+                <cylinder length="0.001" radius="0.0045000000000000005"/>
+            </geometry>
+        </collision>
+        <inertial>
+            <origin rpy="0 1.5707 1.5707" xyz="0 0 0"/>
             <mass value="0.001"/>
             <inertia ixx="5.145833333333334e-09" ixy="0" ixz="0" iyy="5.145833333333334e-09" iyz="0"
@@ -148,5 +148,5 @@
     <link name="front_pitch_link">
         <visual>
-            <origin rpy="0 1.5707 1.5707" xyz="0 0 -0.0005"/>
+            <origin rpy="0 1.5707 1.5707" xyz="0 0 0"/>
             <geometry>
                 <sphere radius="0.0277"/>
@@ -155,5 +155,5 @@
         </visual>
         <collision>
-            <origin rpy="0 1.5707 1.5707" xyz="0 0 -0.0005"/>
+            <origin rpy="0 1.5707 1.5707" xyz="0 0 0"/>
             <geometry>
                 <sphere radius="0.0277"/>
@@ -161,5 +161,5 @@
         </collision>
         <inertial>
-            <origin rpy="0 1.5707 1.5707" xyz="0 0 -0.0005"/>
+            <origin rpy="0 1.5707 1.5707" xyz="0 0 0"/>
             <mass value="0.06"/>
             <inertia ixx="1.8414959999999996e-05" ixy="0.0" ixz="0.0" iyy="1.8414959999999996e-05" iyz="0.0"
@@ -185,18 +185,18 @@
     <link name="back_yaw_link">
         <visual>
-            <origin rpy="0 1.5707 1.5707" xyz="0 0 -0.0005"/>
-            <geometry>
-                <cylinder length="0.001" radius="0.0045000000000000005"/>
-            </geometry>
-            <material name="black"/>
-        </visual>
-        <collision>
-            <origin rpy="0 1.5707 1.5707" xyz="0 0 -0.0005"/>
-            <geometry>
-                <cylinder length="0.001" radius="0.0045000000000000005"/>
-            </geometry>
-        </collision>
-        <inertial>
-            <origin rpy="0 1.5707 1.5707" xyz="0 0 -0.0005"/>
+            <origin rpy="0 1.5707 1.5707" xyz="0.0 0.0 0.0"/>
+            <geometry>
+                <cylinder length="0.001" radius="0.0045000000000000005"/>
+            </geometry>
+            <material name="black"/>
+        </visual>
+        <collision>
+            <origin rpy="0 1.5707 1.5707" xyz="0.0 0.0 0.0"/>
+            <geometry>
+                <cylinder length="0.001" radius="0.0045000000000000005"/>
+            </geometry>
+        </collision>
+        <inertial>
+            <origin rpy="0 1.5707 1.5707" xyz="0.0 0.0 0.0"/>
             <mass value="0.001"/>
             <inertia ixx="5.145833333333334e-09" ixy="0" ixz="0" iyy="5.145833333333334e-09" iyz="0"
@@ -205,5 +205,5 @@
     </link>
     <joint name="back_yaw_joint" type="continuous">
-        <origin rpy="0 0 0" xyz="-0.13 0 0.0005"/>
+        <origin rpy="0 0 0" xyz="-0.13 0 0.0045"/>
         <parent link="main_body_link"/>
         <child link="back_yaw_link"/>
@@ -217,18 +217,18 @@
     <link name="back_roll_link">
         <visual>
-            <origin rpy="0 1.5707 1.5707" xyz="0 0 -0.0005"/>
-            <geometry>
-                <cylinder length="0.001" radius="0.0045000000000000005"/>
-            </geometry>
-            <material name="black"/>
-        </visual>
-        <collision>
-            <origin rpy="0 1.5707 1.5707" xyz="0 0 -0.0005"/>
-            <geometry>
-                <cylinder length="0.001" radius="0.0045000000000000005"/>
-            </geometry>
-        </collision>
-        <inertial>
-            <origin rpy="0 1.5707 1.5707" xyz="0 0 -0.0005"/>
+            <origin rpy="0 1.5707 1.5707" xyz="0 0 0"/>
+            <geometry>
+                <cylinder length="0.001" radius="0.0045000000000000005"/>
+            </geometry>
+            <material name="black"/>
+        </visual>
+        <collision>
+            <origin rpy="0 1.5707 1.5707" xyz="0 0 0"/>
+            <geometry>
+                <cylinder length="0.001" radius="0.0045000000000000005"/>
+            </geometry>
+        </collision>
+        <inertial>
+            <origin rpy="0 1.5707 1.5707" xyz="0 0 0"/>
             <mass value="0.001"/>
             <inertia ixx="5.145833333333334e-09" ixy="0" ixz="0" iyy="5.145833333333334e-09" iyz="0"

File: xacro/wheel.xacro (robot description, xacro)
@@ -4,5 +4,5 @@
     <xacro:property name="wheel_radius" value="0.0352"/>
     <xacro:property name="wheel_origin_raw" value="1.5707"/>
-    <xacro:property name="wheel_origin_z_axis" value="-0.0176"/>
+    <xacro:property name="wheel_origin_z_axis" value="0.0045"/>
     <xacro:macro name="wheel" params="wheel_name">
         <link name="${wheel_name}">
