Commit message: Update two robots xacro files to activate turn and go forward.

File: urdf/barista_robot_model.urdf (robot description, URDF)
Before this commit: robot barista_robot, 14 links, 13 joints
Links:
- link back_pitch_link: mass 0.06 -> 0.05; geometry collision sphere radius=0.025; visual sphere radius=0.025
- link back_roll_link: mass 0.001 -> 0.05; geometry collision cylinder length=0.015 radius=0.02; visual cylinder length=0.015 radius=0.02
- link back_yaw_link: mass 0.001 -> 0.05; geometry collision cylinder length=0.015 radius=0.02; visual cylinder length=0.015 radius=0.02
- link front_pitch_link: mass 0.06 -> 0.05; geometry collision sphere radius=0.025; visual sphere radius=0.025
- link front_roll_link: mass 0.001 -> 0.05; geometry collision cylinder length=0.015 radius=0.02; visual cylinder length=0.015 radius=0.02
- link front_yaw_link: mass 0.001 -> 0.05; geometry collision cylinder length=0.015 radius=0.02; visual cylinder length=0.015 radius=0.02
- link laser_scanner_model: mass 0.5 -> 0.160
- link main_body_link: mass 5 -> 5.0
- link standoff_rods: mass 0.1 -> 0.4
Joints:
- joint back_pitch_joint: limit effort=1000.0 velocity=100.0 -> (none)
- joint back_roll_joint: limit effort=1000.0 velocity=100.0 -> (none)
- joint back_yaw_joint: limit effort=1000.0 velocity=100.0 -> (none); origin xyz=-0.13 0 0.0045 rpy=0 0 0 -> xyz=-0.13 0 -0.079 rpy=0 0 0
- joint base_link_joint: origin xyz=0 0 0 rpy=0 0 0 -> xyz=0 0 0.0 rpy=0 0 0
- joint body_to_standoff_rods_joint: origin xyz=0.0 0.0 0.265 rpy=0 0 0 -> xyz=0.0 0.0 0.1875 rpy=0 0 0
- joint front_pitch_joint: limit effort=1000.0 velocity=100.0 -> (none)
- joint front_roll_joint: limit effort=1000.0 velocity=100.0 -> (none)
- joint front_yaw_joint: limit effort=1000.0 velocity=100.0 -> (none); origin xyz=0.13 0 0.0045 rpy=0 0 0 -> xyz=0.13 0 -0.079 rpy=0 0 0
- joint laser_frame_joint: origin xyz=0.1 0.0 0.176 rpy=0 0 0.0 -> xyz=0.1 0.0 0.0775 rpy=0 0 0
- joint left_wheel_joint: limit effort=1000.0 velocity=100.0 -> effort=10000 velocity=1000.0; origin xyz=0.0 0.1 0.0 rpy=0 0 0 -> xyz=0.0024 0.13 -0.07 rpy=0.0 0.0 0.0
- joint right_wheel_joint: limit effort=1000.0 velocity=100.0 -> effort=10000 velocity=1000.0; origin xyz=0.0 -0.1 0.0 rpy=0 0 0 -> xyz=0.0024 -0.13 -0.07 rpy=0 0 0

File: xacro/barista_robot_model.urdf.xacro (robot description, xacro)
@@ -1,5 +1,4 @@
 <?xml version="1.6"?>
-<robot xmlns:xacro="http://www.ros.org/wiki/xacro" name="barista_robot"
-       xmlns:xsi="http://www.w3.org/2001/XMLSchema-instance"
+<robot xmlns:xacro="http://www.ros.org/wiki/xacro" name="barista_robot" xmlns:xsi="http://www.w3.org/2001/XMLSchema-instance"
        xsi:schemaLocation="http://www.ros.org/wiki/xacro">
     <xacro:property name="robot_name" value="$(arg robot_name)"/>
@@ -10,4 +9,10 @@
         <color rgba="1.0 0.0 0.0 1"/>
     </material>
+    <material name="green_light">
+        <color rgba="0.0 1.0 0.0 1"/>
+    </material>
+    <material name="green_dark">
+        <color rgba="0.0 0.5 0.0 1"/>
+    </material>
     <material name="blue">
         <color rgba="0.0 0.0 1.0 1.0"/>
@@ -21,32 +26,35 @@
     <xacro:if value="${robot_name == 'morty'}">
         <xacro:property name="rviz_color" value="red"/>
+        <xacro:property name="rviz_wheel_color" value="blue"/>
         <xacro:property name="gazebo_color" value="Gazebo/Red"/>
+        <xacro:property name="gazebo_wheel_color" value="Gazebo/Blue"/>
     </xacro:if>
     <xacro:unless value="${robot_name == 'morty'}">
         <xacro:property name="rviz_color" value="blue"/>
+        <xacro:property name="rviz_wheel_color" value="red"/>
         <xacro:property name="gazebo_color" value="Gazebo/Blue"/>
+        <xacro:property name="gazebo_wheel_color" value="Gazebo/Red"/>
     </xacro:unless>
-    <xacro:property name="caster_rviz_color" value="black"/>
-    <xacro:property name="caster_gazebo_color" value="Gazebo/Black"/>
-    <link name="base_link">
-    </link>
+    <xacro:property name="caster_rviz_color" value="green_light"/>
+    <xacro:property name="caster_gazebo_color" value="Gazebo/Yellow"/>
+    <link name="base_link"/>
     <link name="main_body_link">
         <visual>
+            <origin rpy="0 0 0" xyz="0 0 0"/>
             <geometry>
                 <cylinder length="0.155" radius="0.178"/>
             </geometry>
-            <origin xyz="0 0 0.0956" rpy="0 0 0"/>
             <material name="${rviz_color}"/>
         </visual>
         <collision>
+            <origin rpy="0 0 0" xyz="0 0 0"/>
             <geometry>
                 <cylinder length="0.155" radius="0.178"/>
             </geometry>
-            <origin xyz="0 0 0.0956" rpy="0 0 0"/>
-        </collision>
-        <inertial>
-            <mass value="5"/>
-            <origin xyz="0 0 0.0956" rpy="0 0 0"/>
-            <inertia ixx="04961541666666666" ixy="0" ixz="0" iyy="04961541666666666" iyz="0" izz="07920999999999999"/>
+        </collision>
+        <inertial>
+            <mass value="5.0"/>
+            <origin rpy="0 0 0" xyz="0 0 0"/>
+            <inertia ixx="0.049615416666666667" ixy="0.0" ixz="0.0" iyy="0.049615416666666667" iyz="0.0" izz="0.07920999999999999"/>
         </inertial>
     </link>
@@ -55,4 +63,5 @@
         <parent link="base_link"/>
         <child link="main_body_link"/>
+        <axis xyz="0 0 0"/>
     </joint>
     <gazebo reference="main_body_link">
@@ -61,10 +70,8 @@
     <xacro:wheel wheel_name="left_wheel"/>
     <joint name="left_wheel_joint" type="continuous">
-        <origin rpy="0 0 0" xyz="0.0 0.1 0.0"/>
+        <origin rpy="0.0 0.0 0.0" xyz="0.0 0.13 -0.07"/>
         <parent link="main_body_link"/>
         <child link="left_wheel"/>
-        <axis xyz="0 1 0"/>
-        <limit effort="1000.0" velocity="100.0"/>
-        <dynamics damping="0.0" friction="0.1"/>
+        <axis xyz="0 1 0" rpy="0 0 0"/>
     </joint>
     <gazebo reference="left_wheel">
@@ -73,14 +80,12 @@
         <mu1>10.0</mu1>
         <mu2>10.0</mu2>
-        <material>${gazebo_color}</material>
+        <material>${gazebo_wheel_color}</material>
     </gazebo>
     <xacro:wheel wheel_name="right_wheel"/>
     <joint name="right_wheel_joint" type="continuous">
-        <origin rpy="0 0 0" xyz="0.0 -0.1 0.0"/>
+        <origin rpy="0.0 0.0 0.0" xyz="0.0 -0.13 -0.07"/>
         <parent link="main_body_link"/>
         <child link="right_wheel"/>
-        <axis xyz="0 1 0"/>
-        <limit effort="1000.0" velocity="100.0"/>
-        <dynamics damping="0.0" friction="0.1"/>
+        <axis xyz="0 1 0" rpy="0 0 0"/>
     </joint>
     <gazebo reference="right_wheel">
@@ -89,5 +94,5 @@
         <mu1>10.0</mu1>
         <mu2>10.0</mu2>
-        <material>${gazebo_color}</material>
+        <material>${gazebo_wheel_color}</material>
     </gazebo>
     <!-- Casters -->
@@ -97,5 +102,5 @@
             <origin rpy="0 1.5707 1.5707" xyz="0.0 0 0.0"/>
             <geometry>
-                <cylinder length="0.001" radius="0.0045000000000000005"/>
+                <cylinder length="0.015" radius="0.02"/>
             </geometry>
             <material name="${caster_rviz_color}"/>
@@ -104,21 +109,18 @@
             <origin rpy="0 1.5707 1.5707" xyz="0.0 0 0.0"/>
             <geometry>
-                <cylinder length="0.001" radius="0.0045000000000000005"/>
+                <cylinder length="0.015" radius="0.02"/>
             </geometry>
         </collision>
         <inertial>
             <origin rpy="0 1.5707 1.5707" xyz="0.0 0 0.0"/>
-            <mass value="0.001"/>
-            <inertia ixx="5.145833333333334e-09" ixy="0" ixz="0" iyy="5.145833333333334e-09" iyz="0"
-                     izz="1.0125000000000003e-08"/>
+            <mass value="0.05"/>
+            <inertia ixx="5.9375e-06" ixy="0.0" ixz="0.0" iyy="5.9375e-06" iyz="0.0" izz="1e-05"/>
         </inertial>
     </link>
     <joint name="front_yaw_joint" type="continuous">
-        <origin rpy="0 0 0" xyz="0.13 0 0.0045"/>
+        <origin rpy="0 0 0" xyz="0.13 0 -0.079"/>
         <parent link="main_body_link"/>
         <child link="front_yaw_link"/>
         <axis xyz="0 0 1"/>
-        <limit effort="1000.0" velocity="100.0"/>
-        <dynamics damping="0.0" friction="0.1"/>
     </joint>
     <gazebo reference="front_yaw_link">
@@ -129,19 +131,18 @@
             <origin rpy="0 1.5707 1.5707" xyz="0 0 0"/>
             <geometry>
-                <cylinder length="0.001" radius="0.0045000000000000005"/>
-            </geometry>
-            <material name="${caster_rviz_color}"/>
-        </visual>
-        <collision>
-            <origin rpy="0 1.5707 1.5707" xyz="0 0 0"/>
-            <geometry>
-                <cylinder length="0.001" radius="0.0045000000000000005"/>
-            </geometry>
-        </collision>
-        <inertial>
-            <origin rpy="0 1.5707 1.5707" xyz="0 0 0"/>
-            <mass value="0.001"/>
-            <inertia ixx="5.145833333333334e-09" ixy="0" ixz="0" iyy="5.145833333333334e-09" iyz="0"
-                     izz="1.0125000000000003e-08"/>
+                <cylinder length="0.015" radius="0.02"/>
+            </geometry>
+            <material name="${caster_rviz_color}"/>
+        </visual>
+        <collision>
+            <origin rpy="0 1.5707 1.5707" xyz="0 0 0"/>
+            <geometry>
+                <cylinder length="0.015" radius="0.02"/>
+            </geometry>
+        </collision>
+        <inertial>
+            <origin rpy="0 1.5707 1.5707" xyz="0 0 0"/>
+            <mass value="0.05"/>
+            <inertia ixx="5.9375e-06" ixy="0.0" ixz="0.0" iyy="5.9375e-06" iyz="0.0" izz="1e-05"/>
         </inertial>
     </link>
@@ -151,6 +152,4 @@
         <child link="front_roll_link"/>
         <axis xyz="1 0 0"/>
-        <limit effort="1000.0" velocity="100.0"/>
-        <dynamics damping="0.0" friction="0.1"/>
     </joint>
     <gazebo reference="front_roll_link">
@@ -161,19 +160,18 @@
             <origin rpy="0 1.5707 1.5707" xyz="0 0 0"/>
             <geometry>
-                <sphere radius="0.0277"/>
-            </geometry>
-            <material name="${caster_rviz_color}"/>
-        </visual>
-        <collision>
-            <origin rpy="0 1.5707 1.5707" xyz="0 0 0"/>
-            <geometry>
-                <sphere radius="0.0277"/>
-            </geometry>
-        </collision>
-        <inertial>
-            <origin rpy="0 1.5707 1.5707" xyz="0 0 0"/>
-            <mass value="0.06"/>
-            <inertia ixx="1.8414959999999996e-05" ixy="0.0" ixz="0.0" iyy="1.8414959999999996e-05" iyz="0.0"
-                     izz="1.8414959999999996e-05"/>
+                <sphere radius="0.025"/>
+            </geometry>
+            <material name="${caster_rviz_color}"/>
+        </visual>
+        <collision>
+            <origin rpy="0 1.5707 1.5707" xyz="0 0 0"/>
+            <geometry>
+                <sphere radius="0.025"/>
+            </geometry>
+        </collision>
+        <inertial>
+            <origin rpy="0 1.5707 1.5707" xyz="0 0 0"/>
+            <mass value="0.05"/>
+            <inertia ixx="1.2500000000000002e-05" ixy="0.0" ixz="0.0" iyy="1.2500000000000002e-05" iyz="0.0" izz="1.2500000000000002e-05"/>
         </inertial>
     </link>
@@ -190,6 +188,4 @@
         <child link="front_pitch_link"/>
         <axis xyz="0 1 0"/>
-        <limit effort="1000.0" velocity="100.0"/>
-        <dynamics damping="0.0" friction="0.1"/>
     </joint>
     <!-- Caster Wheel Back -->
@@ -198,5 +194,5 @@
             <origin rpy="0 1.5707 1.5707" xyz="0.0 0.0 0.0"/>
             <geometry>
-                <cylinder length="0.001" radius="0.0045000000000000005"/>
+                <cylinder length="0.015" radius="0.02"/>
             </geometry>
             <material name="${caster_rviz_color}"/>
@@ -205,21 +201,18 @@
             <origin rpy="0 1.5707 1.5707" xyz="0.0 0.0 0.0"/>
             <geometry>
-                <cylinder length="0.001" radius="0.0045000000000000005"/>
+                <cylinder length="0.015" radius="0.02"/>
             </geometry>
         </collision>
         <inertial>
             <origin rpy="0 1.5707 1.5707" xyz="0.0 0.0 0.0"/>
-            <mass value="0.001"/>
-            <inertia ixx="5.145833333333334e-09" ixy="0" ixz="0" iyy="5.145833333333334e-09" iyz="0"
-                     izz="1.0125000000000003e-08"/>
+            <mass value="0.05"/>
+            <inertia ixx="5.9375e-06" ixy="0.0" ixz="0.0" iyy="5.9375e-06" iyz="0.0" izz="1e-05"/>
         </inertial>
     </link>
     <joint name="back_yaw_joint" type="continuous">
-        <origin rpy="0 0 0" xyz="-0.13 0 0.0045"/>
+        <origin rpy="0 0 0" xyz="-0.13 0 -0.079"/>
         <parent link="main_body_link"/>
         <child link="back_yaw_link"/>
         <axis xyz="0 0 1"/>
-        <limit effort="1000.0" velocity="100.0"/>
-        <dynamics damping="0.0" friction="0.1"/>
     </joint>
     <gazebo reference="back_yaw_link">
@@ -230,19 +223,18 @@
             <origin rpy="0 1.5707 1.5707" xyz="0 0 0"/>
             <geometry>
-                <cylinder length="0.001" radius="0.0045000000000000005"/>
-            </geometry>
-            <material name="${caster_rviz_color}"/>
-        </visual>
-        <collision>
-            <origin rpy="0 1.5707 1.5707" xyz="0 0 0"/>
-            <geometry>
-                <cylinder length="0.001" radius="0.0045000000000000005"/>
-            </geometry>
-        </collision>
-        <inertial>
-            <origin rpy="0 1.5707 1.5707" xyz="0 0 0"/>
-            <mass value="0.001"/>
-            <inertia ixx="5.145833333333334e-09" ixy="0" ixz="0" iyy="5.145833333333334e-09" iyz="0"
-                     izz="1.0125000000000003e-08"/>
+                <cylinder length="0.015" radius="0.02"/>
+            </geometry>
+            <material name="${caster_rviz_color}"/>
+        </visual>
+        <collision>
+            <origin rpy="0 1.5707 1.5707" xyz="0 0 0"/>
+            <geometry>
+                <cylinder length="0.015" radius="0.02"/>
+            </geometry>
+        </collision>
+        <inertial>
+            <origin rpy="0 1.5707 1.5707" xyz="0 0 0"/>
+            <mass value="0.05"/>
+            <inertia ixx="5.9375e-06" ixy="0.0" ixz="0.0" iyy="5.9375e-06" iyz="0.0" izz="1e-05"/>
         </inertial>
     </link>
@@ -252,6 +244,4 @@
         <child link="back_roll_link"/>
         <axis xyz="1 0 0"/>
-        <limit effort="1000.0" velocity="100.0"/>
-        <dynamics damping="0.0" friction="0.1"/>
     </joint>
     <gazebo reference="back_roll_link">
@@ -262,19 +252,18 @@
             <origin rpy="0 1.5707 1.5707" xyz="0 0 0"/>
             <geometry>
-                <sphere radius="0.0277"/>
-            </geometry>
-            <material name="${caster_rviz_color}"/>
-        </visual>
-        <collision>
-            <origin rpy="0 1.5707 1.5707" xyz="0 0 0"/>
-            <geometry>
-                <sphere radius="0.0277"/>
-            </geometry>
-        </collision>
-        <inertial>
-            <origin rpy="0 1.5707 1.5707" xyz="0 0 0"/>
-            <mass value="0.06"/>
-            <inertia ixx="1.8414959999999996e-05" ixy="0.0" ixz="0.0" iyy="1.8414959999999996e-05" iyz="0.0"
-                     izz="1.8414959999999996e-05"/>
+                <sphere radius="0.025"/>
+            </geometry>
+            <material name="${caster_rviz_color}"/>
+        </visual>
+        <collision>
+            <origin rpy="0 1.5707 1.5707" xyz="0 0 0"/>
+            <geometry>
+                <sphere radius="0.025"/>
+            </geometry>
+        </collision>
+        <inertial>
+            <origin rpy="0 1.5707 1.5707" xyz="0 0 0"/>
+            <mass value="0.05"/>
+            <inertia ixx="1.2500000000000002e-05" ixy="0.0" ixz="0.0" iyy="1.2500000000000002e-05" iyz="0.0" izz="1.2500000000000002e-05"/>
         </inertial>
     </link>
@@ -291,41 +280,40 @@
         <child link="back_pitch_link"/>
         <axis xyz="0 1 0"/>
-        <limit effort="1000.0" velocity="100.0"/>
-        <dynamics damping="0.0" friction="0.1"/>
-    </joint>
-    <!-- standoff_rods -->
-    <link name="standoff_rods">
-        <xacro:standoff x_pos="0.089" y_pos="0.089"/>
-        <xacro:standoff x_pos="-0.089" y_pos="0.089"/>
-        <xacro:standoff x_pos="-0.089" y_pos="-0.089"/>
-        <xacro:standoff x_pos="0.089" y_pos="-0.089"/>
-        <inertial>
-            <mass value="0.1"/>
-            <inertia ixx="0.00040583333333333335" ixy="0" ixz="0" iyy="0.00040583333333333335" iyz="0" izz="5e-06"/>
-        </inertial>
-    </link>
-    <joint name="body_to_standoff_rods_joint" type="fixed">
-        <parent link="main_body_link"/>
-        <child link="standoff_rods"/>
-        <origin xyz="0.0 0.0 0.265" rpy="0 0 0"/>
-    </joint>
-    <xacro:cup_holder_tray/>
-    <joint name="standoff_rods_to_tray_joint" type="fixed">
-        <parent link="standoff_rods"/>
-        <child link="cup_holder"/>
-        <origin xyz="0 0 0.155" rpy="0 0 0"/>
-    </joint>
-    <gazebo reference="cup_holder">
-        <material>${gazebo_color}</material>
-    </gazebo>
-    <!-- Laser scanner (conditional) -->
-    <xacro:arg name="include_laser" default="true"/>
-    <xacro:if value="$(arg include_laser)">
-        <xacro:include filename="$(find barista_robot_description)/xacro/laser_scanner.xacro"/>
-        <xacro:laser_scanner/>
-    </xacro:if>
-    <gazebo reference="laser_scanner_model">
-        <material>${gazebo_color}</material>
-    </gazebo>
+    </joint>
+        <!-- standoff_rods -->
+        <link name="standoff_rods">
+            <xacro:standoff x_pos="0.106" y_pos="0.106"/>
+            <xacro:standoff x_pos="-0.106" y_pos="0.106"/>
+            <xacro:standoff x_pos="-0.106" y_pos="-0.106"/>
+            <xacro:standoff x_pos="0.106" y_pos="-0.106"/>
+            <inertial>
+                <mass value="0.4"/>
+                <origin rpy="0 0 0" xyz="0 0 0"/>
+                <inertia ixx="0.004226666666666668" ixy="0.0" ixz="0.0" iyy="0.0019466666666666666" iyz="0.0" izz="0.002946666666666667"/>
+            </inertial>
+        </link>
+        <joint name="body_to_standoff_rods_joint" type="fixed">
+            <origin rpy="0 0 0" xyz="0.0 0.0 0.1875"/>
+            <parent link="main_body_link"/>
+            <child link="standoff_rods"/>
+        </joint>
+        <xacro:cup_holder_tray/>
+        <joint name="standoff_rods_to_tray_joint" type="fixed">
+            <origin rpy="0 0 0" xyz="0 0 0.155"/>
+            <parent link="standoff_rods"/>
+            <child link="cup_holder"/>
+        </joint>
+        <gazebo reference="cup_holder">
+            <material>${gazebo_color}</material>
+        </gazebo>
+        <!-- Laser scanner (conditional) -->
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
File: xacro/laser_scanner.xacro (robot description, xacro)
@@ -24,5 +24,5 @@
         </link>
         <joint name="laser_frame_joint" type="fixed">
-            <origin xyz="0.1 0.0 0.176" rpy="0 0 0.0"/>
+            <origin xyz="0.1 0.0 0.0775" rpy="0 0 0.0"/>
             <parent link="main_body_link"/>
             <child link="laser_scanner_model"/>

File: xacro/wheel.xacro (robot description, xacro)
@@ -3,10 +3,9 @@
     <xacro:property name="wheel_width" value="0.0206"/>
     <xacro:property name="wheel_radius" value="0.0352"/>
-    <xacro:property name="wheel_origin_raw" value="1.5707"/>
-    <xacro:property name="wheel_origin_z_axis" value="0.0045"/>
+    <xacro:property name="wheel_rotate_90degree" value="1.5707"/>
     <xacro:macro name="wheel" params="wheel_name">
         <link name="${wheel_name}">
             <visual>
-                <origin rpy="${wheel_origin_raw} 0.0 0.0" xyz="0 0 ${wheel_origin_z_axis}"/>
+                <origin rpy="0.0 ${wheel_rotate_90degree} ${wheel_rotate_90degree}" xyz="0 0 0"/>
                 <geometry>
                     <cylinder length="${wheel_width}" radius="${wheel_radius}"/>
@@ -15,5 +14,5 @@
             </visual>
             <collision>
-                <origin rpy="${wheel_origin_raw} 0.0 0.0" xyz="0 0 ${wheel_origin_z_axis}"/>
+                <origin rpy="0.0 ${wheel_rotate_90degree} ${wheel_rotate_90degree}" xyz="0 0 0"/>
                 <geometry>
                     <cylinder length="${wheel_width}" radius="${wheel_radius}"/>
@@ -21,5 +20,5 @@
             </collision>
             <inertial>
-                <origin rpy="${wheel_origin_raw} 0.0 0.0" xyz="0 0 ${wheel_origin_z_axis}"/>
+                <origin rpy="0.0 ${wheel_rotate_90degree} ${wheel_rotate_90degree}" xyz="0 0 0"/>
                 <mass value="0.5"/>
                 <inertia ixx="0.00017256166666666667" ixy="0" ixz="0" iyy="0.00017256166666666667" iyz="0"
