Commit message: Updated to modify robots to move and run

File: xacro/wheel.xacro (robot description, xacro)
@@ -3,17 +3,16 @@
     <xacro:property name="wheel_width" value="0.0206"/>
     <xacro:property name="wheel_radius" value="0.0352"/>
-    <xacro:property name="wheel_origin_raw" value="1.5707"/>
-    <xacro:property name="wheel_origin_z_axis" value="0.0045"/>
+    <xacro:property name="wheel_rotate_90degree" value="1.5707"/>
     <xacro:macro name="wheel" params="wheel_name">
         <link name="${wheel_name}">
             <visual>
-                <origin rpy="${wheel_origin_raw} 0.0 0.0" xyz="0 0 ${wheel_origin_z_axis}"/>
+                <origin rpy="${wheel_rotate_90degree} 0.0 0.0" xyz="0 0 0"/>
                 <geometry>
                     <cylinder length="${wheel_width}" radius="${wheel_radius}"/>
                 </geometry>
-                <material name="${rviz_color}"/>
+                <material name="${rviz_wheel_color}"/>
             </visual>
             <collision>
-                <origin rpy="${wheel_origin_raw} 0.0 0.0" xyz="0 0 ${wheel_origin_z_axis}"/>
+                <origin rpy="${wheel_rotate_90degree} 0.0 0.0" xyz="0 0 0"/>
                 <geometry>
                     <cylinder length="${wheel_width}" radius="${wheel_radius}"/>
@@ -21,8 +20,7 @@
             </collision>
             <inertial>
-                <origin rpy="${wheel_origin_raw} 0.0 0.0" xyz="0 0 ${wheel_origin_z_axis}"/>
+                <origin rpy="${wheel_rotate_90degree} 0.0 0.0" xyz="0 0 0"/>
                 <mass value="0.5"/>
-                <inertia ixx="0.00017256166666666667" ixy="0" ixz="0" iyy="0.00017256166666666667" iyz="0"
-                         izz="0.00030976"/>
+                <inertia ixx="1.7256166666666667e-04" ixy="0.0" ixz="0.0" iyy="1.7256166666666667e-04" iyz="0.0" izz="3.0976e-04"/>
             </inertial>
         </link>
