Commit message: Upload multiple-robots functions

File: xacro/barista_robot_model.urdf.xacro (robot description, xacro)
@@ -3,4 +3,5 @@
        xmlns:xsi="http://www.w3.org/2001/XMLSchema-instance"
        xsi:schemaLocation="http://www.ros.org/wiki/xacro">
+    <xacro:property name="robot_name" value="$(arg robot_name)"/>
     <xacro:include filename="$(find barista_robot_description)/xacro/wheel.xacro"/>
     <xacro:include filename="$(find barista_robot_description)/xacro/standoff.xacro"/>
@@ -18,4 +19,14 @@
         <color rgba="0.0 0.0 0.0 1.0"/>
     </material>
+    <xacro:if value="${robot_name == 'morty'}">
+        <xacro:property name="rviz_color" value="red"/>
+        <xacro:property name="gazebo_color" value="Gazebo/Red"/>
+    </xacro:if>
+    <xacro:unless value="${robot_name == 'morty'}">
+        <xacro:property name="rviz_color" value="blue"/>
+        <xacro:property name="gazebo_color" value="Gazebo/Blue"/>
+    </xacro:unless>
+    <xacro:property name="caster_rviz_color" value="black"/>
+    <xacro:property name="caster_gazebo_color" value="Gazebo/Black"/>
     <link name="base_link">
     </link>
@@ -26,5 +37,5 @@
             </geometry>
             <origin xyz="0 0 0.0956" rpy="0 0 0"/>
-            <material name="blue"/>
+            <material name="${rviz_color}"/>
         </visual>
         <collision>
@@ -46,5 +57,5 @@
     </joint>
     <gazebo reference="main_body_link">
-        <material>Gazebo/Blue</material>
+        <material>${gazebo_color}</material>
     </gazebo>
     <xacro:wheel wheel_name="left_wheel"/>
@@ -62,7 +73,15 @@
         <mu1>10.0</mu1>
         <mu2>10.0</mu2>
-        <material>Gazebo/Red</material>
+        <material>${gazebo_color}</material>
     </gazebo>
     <xacro:wheel wheel_name="right_wheel"/>
+    <joint name="right_wheel_joint" type="continuous">
+        <origin rpy="0 0 0" xyz="0.0 -0.1 0.0"/>
+        <parent link="main_body_link"/>
+        <child link="right_wheel"/>
+        <axis xyz="0 1 0"/>
+        <limit effort="1000.0" velocity="100.0"/>
+        <dynamics damping="0.0" friction="0.1"/>
+    </joint>
     <gazebo reference="right_wheel">
         <kp>1000000000000000000000000000.0</kp>
@@ -70,14 +89,6 @@
         <mu1>10.0</mu1>
         <mu2>10.0</mu2>
-        <material>Gazebo/Red</material>
-    </gazebo>
-    <joint name="right_wheel_joint" type="continuous">
-        <origin rpy="0 0 0" xyz="0.0 -0.1 0.0"/>
-        <parent link="main_body_link"/>
-        <child link="right_wheel"/>
-        <axis xyz="0 1 0"/>
-        <limit effort="1000.0" velocity="100.0"/>
-        <dynamics damping="0.0" friction="0.1"/>
-    </joint>
+        <material>${gazebo_color}</material>
+    </gazebo>
     <!-- Casters -->
     <!-- Caster Wheel Front -->
@@ -88,5 +99,5 @@
                 <cylinder length="0.001" radius="0.0045000000000000005"/>
             </geometry>
-            <material name="black"/>
+            <material name="${caster_rviz_color}"/>
         </visual>
         <collision>
@@ -112,5 +123,5 @@
     </joint>
     <gazebo reference="front_yaw_link">
-        <material>Gazebo/Black</material>
+        <material>${caster_gazebo_color}</material>
     </gazebo>
     <link name="front_roll_link">
@@ -120,5 +131,5 @@
                 <cylinder length="0.001" radius="0.0045000000000000005"/>
             </geometry>
-            <material name="black"/>
+            <material name="${caster_rviz_color}"/>
         </visual>
         <collision>
@@ -144,5 +155,5 @@
     </joint>
     <gazebo reference="front_roll_link">
-        <material>Gazebo/Black</material>
+        <material>${caster_gazebo_color}</material>
     </gazebo>
     <link name="front_pitch_link">
@@ -152,5 +163,5 @@
                 <sphere radius="0.0277"/>
             </geometry>
-            <material name="black"/>
+            <material name="${caster_rviz_color}"/>
         </visual>
         <collision>
@@ -172,5 +183,5 @@
         <mu1>0.5</mu1>
         <mu2>0.5</mu2>
-        <material>Gazebo/Black</material>
+        <material>${caster_gazebo_color}</material>
     </gazebo>
     <joint name="front_pitch_joint" type="continuous">
@@ -189,5 +200,5 @@
                 <cylinder length="0.001" radius="0.0045000000000000005"/>
             </geometry>
-            <material name="black"/>
+            <material name="${caster_rviz_color}"/>
         </visual>
         <collision>
@@ -213,5 +224,5 @@
     </joint>
     <gazebo reference="back_yaw_link">
-        <material>Gazebo/Black</material>
+        <material>${caster_gazebo_color}</material>
     </gazebo>
     <link name="back_roll_link">
@@ -221,5 +232,5 @@
                 <cylinder length="0.001" radius="0.0045000000000000005"/>
             </geometry>
-            <material name="black"/>
+            <material name="${caster_rviz_color}"/>
         </visual>
         <collision>
@@ -245,5 +256,5 @@
     </joint>
     <gazebo reference="back_roll_link">
-        <material>Gazebo/Black</material>
+        <material>${caster_gazebo_color}</material>
     </gazebo>
     <link name="back_pitch_link">
@@ -253,5 +264,5 @@
                 <sphere radius="0.0277"/>
             </geometry>
-            <material name="black"/>
+            <material name="${caster_rviz_color}"/>
         </visual>
         <collision>
@@ -273,5 +284,5 @@
         <mu1>0.5</mu1>
         <mu2>0.5</mu2>
-        <material>Gazebo/Black</material>
+        <material>${caster_gazebo_color}</material>
     </gazebo>
     <joint name="back_pitch_joint" type="continuous">
@@ -306,5 +317,5 @@
     </joint>
     <gazebo reference="cup_holder">
-        <material>Gazebo/Blue</material>
+        <material>${gazebo_color}</material>
     </gazebo>
     <!-- Laser scanner (conditional) -->
@@ -315,11 +326,12 @@
     </xacro:if>
     <gazebo reference="laser_scanner_model">
-        <material>Gazebo/Gray</material>
+        <material>${gazebo_color}</material>
     </gazebo>
     <!-- PLUGINS -->
     <!-- JOINT PUBLISHER -->
     <gazebo>
-        <plugin name="barista_gazebo_robot_joint_state" filename="libgazebo_ros_joint_state_publisher.so">
+        <plugin name="barista_gazebo_${robot_name}_joint_state" filename="libgazebo_ros_joint_state_publisher.so">
             <ros>
+                <namespace>/${robot_name}</namespace>
                 <remapping>~/out:=joint_states</remapping>
             </ros>
@@ -337,5 +349,10 @@
     <!-- Differential drive -->
     <gazebo>
-        <plugin filename="libgazebo_ros_diff_drive.so" name="differential_drive_controller">
+        <plugin filename="libgazebo_ros_diff_drive.so" name="differential_${robot_name}_drive_controller">
+            <!-- namespace for multiple robots from the same model-->
+            <ros>
+                <namespace>/${robot_name}</namespace>
+                <remapping>/cmd_vel:=cmd_vel</remapping>
+            </ros>
             <!-- wheels -->
             <left_joint>left_wheel_joint</left_joint>
@@ -350,6 +367,6 @@
             <publish_odom>true</publish_odom>
             <publish_odom_tf>true</publish_odom_tf>
-            <odometry_frame>odom</odometry_frame>
-            <robot_base_frame>base_link</robot_base_frame>
+            <odometry_frame>${robot_name}/odom</odometry_frame>
+            <robot_base_frame>${robot_name}/base_link</robot_base_frame>
         </plugin>
     </gazebo>

File: xacro/cup_holder_tray.xacro (robot description, xacro)
@@ -10,5 +10,5 @@
                     <cylinder length="${cup_holder_length}" radius="${cup_holder_radius}"/>
                 </geometry>
-                <material name="blue"/>
+                <material name="${rviz_color}"/>
             </visual>
             <collision>

File: xacro/laser_scanner.xacro (robot description, xacro)
@@ -56,10 +56,11 @@
                 <visualize>true</visualize>
                 <update_rate>10.0</update_rate>
-                <plugin name="barista_laser_info" filename="libgazebo_ros_ray_sensor.so">
+                <plugin name="barista_${robot_name}_laser_info" filename="libgazebo_ros_ray_sensor.so">
                     <ros>
-                        <remapping>~/out:=/scan</remapping>
+                        <namespace>/${robot_name}</namespace>
+                        <remapping>~/out:=${robot_name}/scan</remapping>
                     </ros>
                     <output_type>sensor_msgs/LaserScan</output_type>
-                    <frame_name>laser_scan_frame</frame_name>
+                    <frame_name>${robot_name}/laser_scan_frame</frame_name>
                 </plugin>
             </sensor>

File: xacro/wheel.xacro (robot description, xacro)
@@ -12,5 +12,5 @@
                     <cylinder length="${wheel_width}" radius="${wheel_radius}"/>
                 </geometry>
-                <material name="red"/>
+                <material name="${rviz_color}"/>
             </visual>
             <collision>

Commit message: Modify laser color and position

File: xacro/barista_robot_model.urdf.xacro (robot description, xacro)
@@ -314,5 +314,5 @@
         </xacro:if>
         <gazebo reference="laser_scanner_model">
-            <material>${gazebo_color}</material>
+            <material>Gazebo/Gray</material>
         </gazebo>
     <!-- PLUGINS -->

File: xacro/laser_scanner.xacro (robot description, xacro)
@@ -11,18 +11,17 @@
             </visual>
             <collision>
+                <origin rpy="0 0 0" xyz="0 0 0"/>
                 <geometry>
                     <box size="0.05 0.05 0.07"/>
                 </geometry>
-                <origin xyz="-0.00014534209752988105 -4.803507746853085e-19 0.0315145594104885" rpy="0 0 0"/>
             </collision>
             <inertial>
-                <origin xyz="-0.00014534209752988105 -4.803507746853085e-19 0.0315145594104885" rpy="0 0 0"/>
-                <mass value="0.5"/>
-                <inertia ixx="0.0002727493409814312" ixy="2.001660443078184e-20" ixz="1.6939123675595295e-06"
-                         iyy="0.0002741757886259701" iyz="-4.531588429015321e-20" izz="0.00017954959687268426"/>
+                <mass value="0.160"/>
+                <origin rpy="0 0 0" xyz="0 0 0"/>
+                <inertia ixx="9.866666666666669e-05" ixy="0.0" ixz="0.0" iyy="9.866666666666669e-05" iyz="0.0" izz="6.666666666666668e-05"/>
             </inertial>
         </link>
         <joint name="laser_frame_joint" type="fixed">
-            <origin xyz="0.1 0.0 0.176" rpy="0 0 0.0"/>
+            <origin xyz="0.1 0.0 0.0775" rpy="0 0 0.0"/>
             <parent link="main_body_link"/>
             <child link="laser_scanner_model"/>
