Commit message: Modify laser position and color

File: xacro/laser_scanner.xacro (robot description, xacro)
@@ -11,14 +11,13 @@
             </visual>
             <collision>
+                <origin rpy="0 0 0" xyz="0 0 0"/>
                 <geometry>
                     <box size="0.05 0.05 0.07"/>
                 </geometry>
-                <origin xyz="-0.00014534209752988105 -4.803507746853085e-19 0.0315145594104885" rpy="0 0 0"/>
             </collision>
             <inertial>
-                <origin xyz="-0.00014534209752988105 -4.803507746853085e-19 0.0315145594104885" rpy="0 0 0"/>
-                <mass value="0.5"/>
-                <inertia ixx="0.0002727493409814312" ixy="2.001660443078184e-20" ixz="1.6939123675595295e-06"
-                         iyy="0.0002741757886259701" iyz="-4.531588429015321e-20" izz="0.00017954959687268426"/>
+                <mass value="0.160"/>
+                <origin rpy="0 0 0" xyz="0 0 0"/>
+                <inertia ixx="9.866666666666669e-05" ixy="0.0" ixz="0.0" iyy="9.866666666666669e-05" iyz="0.0" izz="6.666666666666668e-05"/>
             </inertial>
         </link>
